File: kicad/INA219AIDCNR.kicad_sch (KiCad schematic)
At the start: 5 parts, among them U1 INA219AxDCN

Commit message: add anotations
Parts:
- renumbered C1 to C3, R2 to R6, R3 to R7, R1 to R8, U1 to U2
Changed lines of the file:
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@@
 		(on_board yes)
 		(dnp no)
-		(property "Reference" "R3"
+		(property "Reference" "R7"
 			(at 152.4 90.1699 0)
 			(effects
@@
 			(project "INA219AIDCNR-breakout"
 				(path "/99399f2a-756c-4718-9b6a-bb37855e6538/82591c7e-40c7-44fc-90aa-28c612ab8916"
-					(reference "R3")
+					(reference "R7")
 					(unit 1)
 				)
@@
 		(dnp no)
 		(fields_autoplaced yes)
-		(property "Reference" "#PWR010"
+		(property "Reference" "#PWR09"
 			(at 130.81 93.98 0)
 			(effects
@@
 			(project "closed-drybox"
 				(path "/99399f2a-756c-4718-9b6a-bb37855e6538/82591c7e-40c7-44fc-90aa-28c612ab8916"
-					(reference "#PWR010")
+					(reference "#PWR09")
 					(unit 1)
 				)
@@
 		(dnp no)
 		(fields_autoplaced yes)
-		(property "Reference" "C1"
+		(property "Reference" "C3"
 			(at 134.62 80.0099 0)
 			(effects
@@
 			(project ""
 				(path "/99399f2a-756c-4718-9b6a-bb37855e6538/82591c7e-40c7-44fc-90aa-28c612ab8916"
-					(reference "C1")
+					(reference "C3")
 					(unit 1)
 				)
@@
 		(dnp no)
 		(fields_autoplaced yes)
-		(property "Reference" "R1"
+		(property "Reference" "R8"
 			(at 97.79 109.2199 0)
 			(effects
@@
 			(project ""
 				(path "/99399f2a-756c-4718-9b6a-bb37855e6538/82591c7e-40c7-44fc-90aa-28c612ab8916"
-					(reference "R1")
+					(reference "R8")
 					(unit 1)
 				)
@@
 		(on_board yes)
 		(dnp no)
-		(property "Reference" "R2"
+		(property "Reference" "R6"
 			(at 143.51 90.1699 0)
 			(effects
@@
 			(project ""
 				(path "/99399f2a-756c-4718-9b6a-bb37855e6538/82591c7e-40c7-44fc-90aa-28c612ab8916"
-					(reference "R2")
+					(reference "R6")
 					(unit 1)
 				)
@@
 		(dnp no)
 		(fields_autoplaced yes)
-		(property "Reference" "#PWR09"
+		(property "Reference" "#PWR010"
 			(at 119.38 152.4 0)
 			(effects
@@
 			(project ""
 				(path "/99399f2a-756c-4718-9b6a-bb37855e6538/82591c7e-40c7-44fc-90aa-28c612ab8916"
-					(reference "#PWR09")
+					(reference "#PWR010")
 					(unit 1)
 				)
@@
 		(dnp no)
 		(fields_autoplaced yes)
-		(property "Reference" "U1"
+		(property "Reference" "U2"
 			(at 121.5233 96.52 0)
 			(effects
@@
 			(project "INA219AIDCNR-breakout"
 				(path "/99399f2a-756c-4718-9b6a-bb37855e6538/82591c7e-40c7-44fc-90aa-28c612ab8916"
-					(reference "U1")
-					(unit 1)
-				)
+					(reference "U2")
+					(unit 1)
+				)

Commit message: add PCB
Parts:
- renumbered C3 to C7, U2 to U3
Changed lines of the file:
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@@
 		(dnp no)
 		(fields_autoplaced yes)
-		(property "Reference" "#PWR09"
+		(property "Reference" "#PWR014"
 			(at 130.81 93.98 0)
 			(effects
@@
 			(project "closed-drybox"
 				(path "/99399f2a-756c-4718-9b6a-bb37855e6538/82591c7e-40c7-44fc-90aa-28c612ab8916"
-					(reference "#PWR09")
+					(reference "#PWR014")
 					(unit 1)
 				)
@@
 		(dnp no)
 		(fields_autoplaced yes)
-		(property "Reference" "C3"
+		(property "Reference" "C7"
 			(at 134.62 80.0099 0)
 			(effects
@@
 			(project ""
 				(path "/99399f2a-756c-4718-9b6a-bb37855e6538/82591c7e-40c7-44fc-90aa-28c612ab8916"
-					(reference "C3")
+					(reference "C7")
 					(unit 1)
 				)
@@
 		(dnp no)
 		(fields_autoplaced yes)
-		(property "Reference" "#PWR010"
+		(property "Reference" "#PWR015"
 			(at 119.38 152.4 0)
 			(effects
@@
 			(project ""
 				(path "/99399f2a-756c-4718-9b6a-bb37855e6538/82591c7e-40c7-44fc-90aa-28c612ab8916"
-					(reference "#PWR010")
+					(reference "#PWR015")
 					(unit 1)
 				)
@@
 		(dnp no)
 		(fields_autoplaced yes)
-		(property "Reference" "U2"
+		(property "Reference" "U3"
 			(at 121.5233 96.52 0)
 			(effects
@@
 			(project "INA219AIDCNR-breakout"
 				(path "/99399f2a-756c-4718-9b6a-bb37855e6538/82591c7e-40c7-44fc-90aa-28c612ab8916"
-					(reference "U2")
-					(unit 1)
-				)
+					(reference "U3")
+					(unit 1)
+				)

Commit message: update schematic
Parts:
- renumbered R6 to R1, R7 to R2, R8 to R3
Other:
- title: (none) -> closed-drybox
Changed lines of the file:
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@@
 	(generator_version "9.0")
 	(paper "A4")
+	(title_block
+		(title "closed-drybox")
+		(rev "1")
+		(comment 1 "https://github.com/lukstruck/closed-drybox#")
+	)
 	(junction
 		(at 149.86 106.68)
@@
 		(on_board yes)
 		(dnp no)
-		(property "Reference" "R7"
+		(property "Reference" "R2"
 			(at 152.4 90.1699 0)
 			(effects
@@
 			(project "INA219AIDCNR-breakout"
 				(path "/99399f2a-756c-4718-9b6a-bb37855e6538/82591c7e-40c7-44fc-90aa-28c612ab8916"
-					(reference "R7")
+					(reference "R2")
 					(unit 1)
 				)
@@
 		(dnp no)
 		(fields_autoplaced yes)
-		(property "Reference" "#PWR014"
+		(property "Reference" "#PWR011"
 			(at 130.81 93.98 0)
 			(effects
@@
 			(project "closed-drybox"
 				(path "/99399f2a-756c-4718-9b6a-bb37855e6538/82591c7e-40c7-44fc-90aa-28c612ab8916"
-					(reference "#PWR014")
+					(reference "#PWR011")
 					(unit 1)
 				)
@@
 		(dnp no)
 		(fields_autoplaced yes)
-		(property "Reference" "R8"
+		(property "Reference" "R3"
 			(at 97.79 109.2199 0)
 			(effects
@@
 			(project ""
 				(path "/99399f2a-756c-4718-9b6a-bb37855e6538/82591c7e-40c7-44fc-90aa-28c612ab8916"
-					(reference "R8")
+					(reference "R3")
 					(unit 1)
 				)
@@
 		(on_board yes)
 		(dnp no)
-		(property "Reference" "R6"
+		(property "Reference" "R1"
 			(at 143.51 90.1699 0)
 			(effects
@@
 			(project ""
 				(path "/99399f2a-756c-4718-9b6a-bb37855e6538/82591c7e-40c7-44fc-90aa-28c612ab8916"
-					(reference "R6")
+					(reference "R1")
 					(unit 1)
 				)
@@
 		(dnp no)
 		(fields_autoplaced yes)
-		(property "Reference" "#PWR015"
+		(property "Reference" "#PWR012"
 			(at 119.38 152.4 0)
 			(effects
@@
 			(project ""
 				(path "/99399f2a-756c-4718-9b6a-bb37855e6538/82591c7e-40c7-44fc-90aa-28c612ab8916"
-					(reference "#PWR015")
-					(unit 1)
-				)
+					(reference "#PWR012")
+					(unit 1)
+				)
