File: kicad/INA219AIDCNR.kicad_sch (KiCad schematic)
At the start: 5 parts, among them U3 INA219AxDCN

Commit message: set LCSC ID's
Parts:
- C7: LCSC C14663 -> C1591
Changed lines of the file:
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@@
 			)
 		)
-		(property "LCSC" "C14663"
+		(property "LCSC" "C1591"
 			(at 134.62 80.0099 0)
 			(effects
