File: kicad/closed-drybox.kicad_pcb (KiCad board)
At the start: 4 copper layers, 70 x 80 mm, 69 parts, among them J1 Conn_01x02, J10 Conn_01x01_Pin, J11 Conn_01x03_Pin, J2 Power_Jack, J3 Conn_01x02_Pin, J4 Conn_01x02_Pin, J5 Conn_01x02_Pin, J6 Conn_01x05_Pin, J7 Conn_01x04, J8 Conn_01x04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

Commit message: fix vias too close to each other
Routing:
- net +12V: vias 20 -> 18
Changed lines of the file:
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@@
 	)
 	(segment
-		(start 203.5 112.5)
+		(start 203.5 112.200003)
 		(end 203.5 113)
 		(width 1.5)
@@
 	)
 	(segment
-		(start 203.5 111.5)
-		(end 203.5 112)
+		(start 203.5 111.200003)
+		(end 203.5 110.5)
 		(width 1.5)
 		(layer "F.Cu")
@@
 		(start 177.4 111)
 		(end 179.2 111)
-		(width 1.5)
-		(layer "F.Cu")
-		(net 3)
-	)
-	(segment
-		(start 203.5 110.5)
-		(end 203.5 111)
 		(width 1.5)
 		(layer "F.Cu")
@@
 	)
 	(segment
-		(start 203.5 112)
-		(end 203.5 112.5)
-		(width 1.5)
-		(layer "F.Cu")
-		(net 3)
-	)
-	(segment
 		(start 203.5 113)
 		(end 203.75 113)
@@
 	)
 	(segment
-		(start 203.5 111)
-		(end 203.5 111.5)
-		(width 1.5)
-		(layer "F.Cu")
-		(net 3)
-	)
-	(segment
 		(start 197.4 98.975)
 		(end 196.825 98.975)
@@
 	)
 	(segment
+		(start 203.5 111.200003)
+		(end 203.5 112.200003)
+		(width 1.5)
+		(layer "F.Cu")
+		(net 3)
+	)
+	(segment
 		(start 173.2 104.15)
 		(end 174.85 104.15)
@@
 	)
 	(via
-		(at 203.5 112.5)
-		(size 0.6)
-		(drill 0.3)
-		(layers "F.Cu" "B.Cu")
-		(net 3)
-	)
-	(via
-		(at 203.5 112)
+		(at 203.5 112.200003)
 		(size 0.6)
 		(drill 0.3)
@@
 	)
 	(via
-		(at 203.5 111)
-		(size 0.6)
-		(drill 0.3)
-		(layers "F.Cu" "B.Cu")
-		(net 3)
-	)
-	(via
 		(at 198.6 98.975)
 		(size 0.6)
@@
 	)
 	(via
-		(at 203.5 111.5)
-		(size 0.6)
-		(drill 0.3)
+		(at 203.5 111.200003)
+		(size 0.6)
+		(drill 0.3)

Commit message: add GND vias arround caps (next to LDO)
Routing:
- net GND: vias 426 -> 430
Changed lines of the file:
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@@
+	)
+	(via
+		(at 211.15 94.63)
+		(size 0.6)
+		(drill 0.3)
+		(layers "F.Cu" "B.Cu")
+		(free yes)
+		(net 2)
 	)
 	(via
@@
 	)
 	(via
+		(at 201.44 96.73)
+		(size 0.6)
+		(drill 0.3)
+		(layers "F.Cu" "B.Cu")
+		(free yes)
+		(net 2)
+	)
+	(via
 		(at 170.18 47.963137)
 		(size 0.6)
@@
 	)
 	(via
+		(at 214.46 94.48)
+		(size 0.6)
+		(drill 0.3)
+		(layers "F.Cu" "B.Cu")
+		(free yes)
+		(net 2)
+	)
+	(via
 		(at 227 106.6)
 		(size 0.6)
@@
 		(size 0.6)
 		(drill 0.3)
+		(layers "F.Cu" "B.Cu")
+		(free yes)
+		(net 2)
+	)
+	(via
+		(at 199.82 96.67)
+		(size 0.6)
+		(drill 0.3)

Commit message: 3.3V LDO
Parts:
- U1: value AMS1117-5.0 -> AMS1117-3.3
Changed lines of the file:
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@@
 			)
 		)
-		(property "Value" "AMS1117-5.0"
+		(property "Value" "AMS1117-3.3"
 			(at 0.4 4.4 0)
 			(layer "F.SilkS")
@@
 			)
 		)
-		(property "Description" "1A Low Dropout regulator, positive, 5.0V fixed output, SOT-223"
+		(property "Description" "1A Low Dropout regulator, positive, 3.3V fixed output, SOT-223"
 			(at 0 0 0)
 			(unlocked yes)
@@
 		(layer "Edge.Cuts")
 	)
-	(gr_text "GND"
-		(at 196.5 60 0)
+	(gr_text "SCL"
+		(at 196.5 57.5 0)
 		(layer "F.SilkS")
 		(effects
@@
 		)
 	)
-	(gr_text "3.3V"
-		(at 213.4 60.2 0)
+	(gr_text "GND"
+		(at 196.5 60 0)
 		(layer "F.SilkS")
 		(effects
@@
 		)
 	)
-	(gr_text "3"
-		(at 220.7 60 0)
+	(gr_text "SDA"
+		(at 196.5 62.5 0)
 		(layer "F.SilkS")
 		(effects
@@
 		)
 	)
-	(gr_text "GND"
-		(at 213.4 57.6 0)
+	(gr_text "3.3V"
+		(at 196.5 65 0)
 		(layer "F.SilkS")
 		(effects
@@
 		)
 	)
-	(gr_text "T"
-		(at 220.7 62.5 0)
+	(gr_text "SDA"
+		(at 212.4 62.6 0)
 		(layer "F.SilkS")
 		(effects
@@
 		)
 	)
-	(gr_text "SDA"
-		(at 212.4 62.6 0)
+	(gr_text "SCL"
+		(at 212.5 65.25 0)
 		(layer "F.SilkS")
 		(effects
@@
 		)
 	)
-	(gr_text "SCL"
-		(at 212.5 65.25 0)
+	(gr_text "GND"
+		(at 213.4 57.6 0)
 		(layer "F.SilkS")
 		(effects
@@
 		)
 	)
-	(gr_text "SCL"
-		(at 196.5 57.5 0)
+	(gr_text "3.3V"
+		(at 213.4 60.2 0)
 		(layer "F.SilkS")
 		(effects
@@
 		)
 	)
-	(gr_text "3.3V"
-		(at 196.5 65 0)
+	(gr_text "G"
+		(at 220.7 57.75 0)
 		(layer "F.SilkS")
 		(effects
@@
 		)
 	)
-	(gr_text "SDA"
-		(at 196.5 62.5 0)
+	(gr_text "3"
+		(at 220.7 60 0)
 		(layer "F.SilkS")
 		(effects
@@
 		)
 	)
-	(gr_text "G"
-		(at 220.7 57.75 0)
+	(gr_text "T"
+		(at 220.7 62.5 0)
 		(layer "F.SilkS")
 		(effects
@@
 		)
 	)
-	(gr_text "{\n  \"ViaStitching\": \"0.2\",\n  \"GND\": {\n    \"HSpacing\": \"2.5\",\n    \"VSpacing\": \"2.5\",\n    \"HOffset\": \"0\",\n    \"VOffset\": \"0\",\n    \"Clearance\": \"2\",\n    \"Randomize\": false\n  }\n}"
+	(gr_text "{\n  \"ViaStitching\": \"0.2\",\n  \"GND\": {\n    \"HSpacing\": \"0.5\",\n    \"VSpacing\": \"0.5\",\n    \"HOffset\": \"0\",\n    \"VOffset\": \"0\",\n    \"Clearance\": \"0.2\",\n    \"Randomize\": false\n  }\n}"
 		(at 0 0 0)
 		(layer "User.9")
@@
 		)
 	)
-	(gr_text "{\n  \"ViaStitching\": \"0.2\",\n  \"GND\": {\n    \"HSpacing\": \"2\",\n    \"VSpacing\": \"2\",\n    \"HOffset\": \"0\",\n    \"VOffset\": \"0\",\n    \"Clearance\": \"0\",\n    \"Randomize\": false\n  }\n}"
+	(gr_text "{\n  \"ViaStitching\": \"0.2\",\n  \"GND\": {\n    \"HSpacing\": \"1\",\n    \"VSpacing\": \"1\",\n    \"HOffset\": \"0\",\n    \"VOffset\": \"0\",\n    \"Clearance\": \"0\",\n    \"Randomize\": false\n  }\n}"
 		(at 0 0 0)
 		(layer "User.9")
@@
 		)
 	)
-	(gr_text "{\n  \"ViaStitching\": \"0.2\",\n  \"GND\": {\n    \"HSpacing\": \"0.5\",\n    \"VSpacing\": \"0.5\",\n    \"HOffset\": \"0\",\n    \"VOffset\": \"0\",\n    \"Clearance\": \"0.2\",\n    \"Randomize\": false\n  }\n}"
+	(gr_text "{\n  \"ViaStitching\": \"0.2\",\n  \"GND\": {\n    \"HSpacing\": \"1\",\n    \"VSpacing\": \"1\",\n    \"HOffset\": \"0\",\n    \"VOffset\": \"0\",\n    \"Clearance\": \"0.3\",\n    \"Randomize\": false\n  }\n}"
 		(at 0 0 0)
 		(layer "User.9")
@@
 		)
 	)
-	(gr_text "{\n  \"ViaStitching\": \"0.2\",\n  \"GND\": {\n    \"HSpacing\": \"2.5\",\n    \"VSpacing\": \"2.5\",\n    \"HOffset\": \"0\",\n    \"VOffset\": \"0\",\n    \"Clearance\": \"2\",\n    \"Randomize\": false\n  }\n}"
+	(gr_text "{\n  \"ViaStitching\": \"0.2\",\n  \"GND\": {\n    \"HSpacing\": \"2\",\n    \"VSpacing\": \"2\",\n    \"HOffset\": \"0\",\n    \"VOffset\": \"0\",\n    \"Clearance\": \"0\",\n    \"Randomize\": false\n  }\n}"
 		(at 0 0 0)
 		(layer "User.9")
@@
 		)
 	)
-	(gr_text "{\n  \"ViaStitching\": \"0.2\",\n  \"GND\": {\n    \"HSpacing\": \"2.5\",\n    \"VSpacing\": \"2.5\",\n    \"HOffset\": \"0\",\n    \"VOffset\": \"0\",\n    \"Clearance\": \"2\",\n    \"Randomize\": false\n  }\n}"
-		(at 0 0 0)
-		(layer "User.9")
-		(effects
-			(font
-				(size 1.27 1.27)
-			)
-			(justify left top)
-		)
-	)
-	(gr_text "{\n  \"ViaStitching\": \"0.2\",\n  \"GND\": {\n    \"HSpacing\": \"3\",\n    \"VSpacing\": \"3\",\n    \"HOffset\": \"0\",\n    \"VOffset\": \"0\",\n    \"Clearance\": \"2\",\n    \"Randomize\": false\n  }\n}"
-		(at 0 0 0)
-		(layer "User.9")
-		(effects
-			(font
-				(size 1.27 1.27)
-			)
-			(justify left top)
-		)
-	)
 	(gr_text "{\n  \"ViaStitching\": \"0.2\",\n  \"GND\": {\n    \"HSpacing\": \"3\",\n    \"VSpacing\": \"3\",\n    \"HOffset\": \"0\",\n    \"VOffset\": \"0\",\n    \"Clearance\": \"2\",\n    \"Randomize\": false\n  }\n}"
 		(at 0 0 0)
 		(layer "User.9")
-		(effects
-			(font
-				(size 1.27 1.27)
-			)
-			(justify left top)
-		)
-	)
-	(gr_text "{\n  \"ViaStitching\": \"0.2\",\n  \"GND\": {\n    \"HSpacing\": \"1\",\n    \"VSpacing\": \"1\",\n    \"HOffset\": \"0\",\n    \"VOffset\": \"0\",\n    \"Clearance\": \"0\",\n    \"Randomize\": false\n  }\n}"
-		(at 0 0 0)
-		(layer "User.9")
-		(effects
-			(font
-				(size 1.27 1.27)
-			)
-			(justify left top)
-		)
-	)
-	(gr_text "{\n  \"ViaStitching\": \"0.2\",\n  \"GND\": {\n    \"HSpacing\": \"1\",\n    \"VSpacing\": \"1\",\n    \"HOffset\": \"0\",\n    \"VOffset\": \"0\",\n    \"Clearance\": \"0\",\n    \"Randomize\": false\n  }\n}"
-		(at 0 0 0)
-		(layer "User.9")
-		(effects
-			(font
-				(size 1.27 1.27)
-			)
-			(justify left top)
-		)
-	)
-	(gr_text "{\n  \"ViaStitching\": \"0.2\",\n  \"GND\": {\n    \"HSpacing\": \"1\",\n    \"VSpacing\": \"1\",\n    \"HOffset\": \"0\",\n    \"VOffset\": \"0\",\n    \"Clearance\": \"0.3\",\n    \"Randomize\": false\n  }\n}"
-		(at 0 0 0)
-		(layer "User.9")
