File: kicad/heater.kicad_sch (KiCad schematic)
At the start: 5 parts, among them Q1 AO3400A

Commit message: set LCSC ID's
Parts:
- R4: LCSC C158012 -> C157931
Changed lines of the file:
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@@
 			)
 		)
-		(property "LCSC" "C158012"
+		(property "LCSC" "C157931"
 			(at 93.98 73.6599 0)
 			(effects
